Commit message: Update goliath_description.urdf

File: goliath_description.urdf (robot description, URDF)
Before this commit: robot goliath, 6 links, 5 joints
Links:
- removed link end_effector
- removed link link1
- removed link link2
- removed link link3
- removed link link4
- added link grip_mount_1, mass 0.026038448039166225; collision mesh filename=@viththagi/viththagi.github.io/mesh/grip_mount_1.stl scale=0.001 0.001 0.001; visual mesh filename=@viththagi/viththagi.github.io/mesh/grip_mount_1.stl scale=0.001 0.001 0.001
- added link left_mount_1, mass 0.005850260501194334; collision mesh filename=@viththagi/viththagi.github.io/mesh/left_mount_1.stl scale=0.001 0.001 0.001; visual mesh filename=@viththagi/viththagi.github.io/mesh/left_mount_1.stl scale=0.001 0.001 0.001
- added link link_1, mass 3.0; collision mesh filename=@viththagi/viththagi.github.io/mesh/link_1.stl; visual mesh filename=@viththagi/viththagi.github.io/mesh/link_1.stl
- added link link_2, mass 2.5; collision mesh filename=@viththagi/viththagi.github.io/mesh/link_2.stl; visual mesh filename=@viththagi/viththagi.github.io/mesh/link_2.stl
- added link link_3, mass 2.0; collision mesh filename=@viththagi/viththagi.github.io/mesh/link_3.stl; visual mesh filename=@viththagi/viththagi.github.io/mesh/link_3.stl
- added link link_4, mass 1.5; collision mesh filename=@viththagi/viththagi.github.io/mesh/link_4.stl; visual mesh filename=@viththagi/viththagi.github.io/mesh/link_4.stl
- added link link_5, mass 1.2; collision mesh filename=@viththagi/viththagi.github.io/mesh/link_5.stl; visual mesh filename=@viththagi/viththagi.github.io/mesh/link_5.stl
- added link link_6, mass 0.8; collision mesh filename=@viththagi/viththagi.github.io/mesh/tool_connector.stl; visual mesh filename=@viththagi/viththagi.github.io/mesh/tool_connector.stl
- added link power_box, mass 1.0; collision mesh filename=@viththagi/viththagi.github.io/mesh/power_box.stl; visual mesh filename=@viththagi/viththagi.github.io/mesh/power_box.stl
- added link right_mount_1, mass 0.005851464483284041; collision mesh filename=@viththagi/viththagi.github.io/mesh/right_mount_1.stl scale=0.001 0.001 0.001; visual mesh filename=@viththagi/viththagi.github.io/mesh/right_mount_1.stl scale=0.001 0.001 0.001
- added link rubber_left_1, mass 0.008265327612092782; collision mesh filename=@viththagi/viththagi.github.io/mesh/rubber_left_1.stl scale=0.001 0.001 0.001; visual mesh filename=@viththagi/viththagi.github.io/mesh/rubber_left_1.stl scale=0.001 0.001 0.001
- added link rubber_right_1, mass 0.008265327612092756; collision mesh filename=@viththagi/viththagi.github.io/mesh/rubber_right_1.stl scale=0.001 0.001 0.001; visual mesh filename=@viththagi/viththagi.github.io/mesh/rubber_right_1.stl scale=0.001 0.001 0.001
- added link t_shirt_1, mass 0.0026146856075812087; collision mesh filename=@viththagi/viththagi.github.io/mesh/t_shirt_1.stl scale=0.001 0.001 0.001; visual mesh filename=@viththagi/viththagi.github.io/mesh/t_shirt_1.stl scale=0.001 0.001 0.001
- added link tool_base, mass 0.3; collision mesh filename=@viththagi/viththagi.github.io/mesh/tool_base.stl; visual mesh filename=@viththagi/viththagi.github.io/mesh/tool_base.stl
- added link tool_connector, mass 0.5; collision mesh filename=@viththagi/viththagi.github.io/mesh/tool_base.stl; visual mesh filename=@viththagi/viththagi.github.io/mesh/tool_base.stl
- added link world
- link base_link: geometry collision mesh filename=@viththagi/viththagi.github.io/mesh/link_0.stl; visual mesh filename=@viththagi/viththagi.github.io/mesh/link_0.stl
Joints:
- removed joint joint1
- removed joint joint2
- removed joint joint3
- removed joint joint4
- removed joint joint5
- added joint Rigid_20: type fixed, parent tool_base, child grip_mount_1, origin xyz=0.000365 -0.006365 0.008562 rpy=0 0 0
- added joint Rigid_24: type fixed, parent left_mount_1, child rubber_left_1, origin xyz=-0.01514 0.01049 0.027691 rpy=0 0 0
- added joint Rigid_25: type fixed, parent right_mount_1, child rubber_right_1, origin xyz=0.01418 0.0105 0.028237 rpy=0 0 0
- added joint Rigid_26: type fixed, parent grip_mount_1, child t_shirt_1, origin xyz=-0.000556 -0.001302 0.013562 rpy=0 0 0
- added joint Slider_22: type prismatic, parent t_shirt_1, child left_mount_1, origin xyz=-0.022607 -0.008412 0.010565 rpy=0 0 0, axis 0.817033 -0.0 0.576591, limit lower=-0.003 upper=0.022 effort=100 velocity=100
- added joint Slider_23: type prismatic, parent t_shirt_1, child right_mount_1, origin xyz=0.022917 -0.008412 0.010857 rpy=0 0 0, axis 0.820609 0.0 -0.57149, limit lower=-0.022 upper=0.003 effort=100 velocity=100
- added joint base_joint: type fixed, parent world, child base_link, origin xyz=0 0 0 rpy=0 0 0, axis 0 0 1
- added joint joint_1: type revolute, parent base_link, child link_1, origin xyz=0 0 0.104 rpy=0 0 0, axis 0 0 1, limit lower=-3.14159 upper=3.14159 effort=1000.0 velocity=2.5
- added joint joint_2: type revolute, parent link_1, child link_2, origin xyz=0 -0.060768 0.1694 rpy=-1.5708 -1.5708 3.14159, axis 0 0 1, limit lower=-1.5708 upper=1.5708 effort=1000.0 velocity=2.5
- added joint joint_3: type revolute, parent link_2, child link_3, origin xyz=0.315 0 -0.0198 rpy=0 3.14159 0, axis 0 0 1, limit lower=-2.6180 upper=2.6180 effort=1000.0 velocity=2.5
- added joint joint_4: type revolute, parent link_3, child link_4, origin xyz=0.066258 0 0.036577 rpy=0 1.5708 0, axis 0 0 1, limit lower=-3.14159 upper=3.14159 effort=1000.0 velocity=2.5
- added joint joint_5: type revolute, parent link_4, child link_5, origin xyz=0.02456 0 -0.319213 rpy=0 1.5708 3.14159, axis 0 0 1, limit lower=-2.0944 upper=2.0944 effort=1000.0 velocity=2.5
- added joint joint_6: type revolute, parent link_5, child link_6, origin xyz=0.07318 0 0.02 rpy=0 1.5708 0, axis 0 0 1, limit lower=-3.14159 upper=3.14159 effort=1000.0 velocity=2.5
- added joint joint_connector_frame: type fixed, parent tool_connector, child tool_base, origin xyz=-0.0038 0.005 0.017 rpy=0 0 0
- added joint joint_powebox: type fixed, parent link_2, child power_box, origin xyz=-0.276 0 -0.057 rpy=0 1.5775 0
- added joint joint_tool_connector_frame: type fixed, parent link_6, child tool_connector, origin xyz=0 0 0 rpy=0 0 0
